Commit message: version up for noetic / ros1 bridge

File: serving_mobile/servingbot_description/urdf/servingbot3.urdf.xacro (robot description, xacro)
@@ -1,4 +1,5 @@
 <?xml version="1.0" ?>
-<robot name="servingbot" xmlns:xacro="http://ros.org/wiki/xacro">
+<robot name="servingbot"
+  xmlns:xacro="http://ros.org/wiki/xacro">
   <xacro:include filename="$(find servingbot_description)/urdf/common_properties.xacro"/>
   <xacro:include filename="$(find servingbot_description)/urdf/servingbot.gazebo.xacro"/>
@@ -9,41 +10,23 @@
     <origin xyz="0.0 0.0 0.2465" rpy="0 0 0"/>
   </joint>
-  <link
-    name="base_link">
-    <inertial>
-      <origin
-        xyz="-0.0070361 -0.0010307 -0.094165"
-        rpy="0 0 0" />
-      <mass
-        value="7" />
-      <inertia
-        ixx="0.114"
-        ixy="3.4187E-05"
-        ixz="-0.0079587"
-        iyy="0.084746"
-        iyz="-0.00069939"
-        izz="0.14914" />
-    </inertial>
-    <visual>
-      <origin
-        xyz="0 0 0"
-        rpy="0 0 0" />
-      <geometry>
-        <mesh
-          filename="package://servingbot_description/meshes/body.STL" />
-      </geometry>
-      <material
-        name="">
-        <color
-          rgba="0.79216 0.81961 0.93333 1" />
-      </material>
-    </visual>
-    <collision>
-      <origin
-        xyz="0 0 0"
-        rpy="0 0 0" />
-      <geometry>
-        <mesh
-          filename="package://servingbot_description/meshes/body.STL" />
+  <link name="base_link">
+    <inertial>
+      <origin xyz="-0.0070361 -0.0010307 -0.094165" rpy="0 0 0" />
+      <mass value="7" />
+      <inertia ixx="0.114" ixy="3.4187E-05" ixz="-0.0079587" iyy="0.084746" iyz="-0.00069939" izz="0.14914" />
+    </inertial>
+    <visual>
+      <origin xyz="0 0 0" rpy="0 0 0" />
+      <geometry>
+        <mesh filename="package://servingbot_description/meshes/body.STL" />
+      </geometry>
+      <material name="">
+        <color rgba="0.79216 0.81961 0.93333 1" />
+      </material>
+    </visual>
+    <collision>
+      <origin xyz="0 0 0" rpy="0 0 0" />
+      <geometry>
+        <mesh filename="package://servingbot_description/meshes/body.STL" />
       </geometry>
     </collision>
@@ -55,15 +38,12 @@
         <mesh filename="package://servingbot_description/meshes/base_plate.STL" />
       </geometry>
-      <material
-        name="">
-        <color
-          rgba="0.79216 0.81961 0.93333 1" />
-      </material>
-    </visual>
-    <collision>
-      <origin xyz="0 0 0" rpy="0 0 0"/>
-      <geometry>
-        <mesh
-          filename="package://servingbot_description/meshes/base_plate.STL" />
+      <material name="">
+        <color rgba="0.79216 0.81961 0.93333 1" />
+      </material>
+    </visual>
+    <collision>
+      <origin xyz="0 0 0" rpy="0 0 0"/>
+      <geometry>
+        <mesh filename="package://servingbot_description/meshes/base_plate.STL" />
       </geometry>
     </collision>
@@ -71,21 +51,12 @@
       <origin xyz="-0.0036904 0 0.0025" rpy="0 0 0"/>
       <mass value="2"/>
-      <inertia ixx="0" ixy="0" ixz="0"
-               iyy="0" iyz="0"
-               izz="0" />
-    </inertial>
-  </link>
-  <joint
-    name="body_joint"
-    type="fixed">
-    <origin
-      xyz="0.0039057 0 -0.08"
-      rpy="-6.913E-15 -1.1102E-16 -5.4234E-31" />
-    <parent
-      link="base_link" />
-    <child
-      link="body_link" />
-    <axis
-      xyz="0 0 0" />
+      <inertia ixx="0" ixy="0" ixz="0" iyy="0" iyz="0" izz="0" />
+    </inertial>
+  </link>
+  <joint name="body_joint" type="fixed">
+    <origin xyz="0.0039057 0 -0.08" rpy="-6.913E-15 -1.1102E-16 -5.4234E-31" />
+    <parent link="base_link" />
+    <child link="body_link" />
+    <axis xyz="0 0 0" />
   </joint>
   <joint name="wheel_left_joint" type="continuous">
@@ -101,15 +72,12 @@
         <mesh filename="package://servingbot_description/meshes/left_wheel.STL" />
       </geometry>
-      <material
-        name="">
-        <color
-          rgba="0.79216 0.81961 0.93333 1" />
-      </material>
-    </visual>
-    <collision>
-      <origin xyz="0 0 0" rpy="0 0 0"/>
-      <geometry>
-        <mesh
-          filename="package://servingbot_description/meshes/left_wheel.STL" />
+      <material name="">
+        <color rgba="0.79216 0.81961 0.93333 1" />
+      </material>
+    </visual>
+    <collision>
+      <origin xyz="0 0 0" rpy="0 0 0"/>
+      <geometry>
+        <mesh filename="package://servingbot_description/meshes/left_wheel.STL" />
       </geometry>
     </collision>
@@ -117,8 +85,6 @@
       <origin xyz="0 0 0" />
       <mass value="3.5" />
-      <inertia ixx="0" ixy="0" ixz="0"
-               iyy="0" iyz="0"
-               izz="0" />
-      </inertial>
+      <inertia ixx="0" ixy="0" ixz="0" iyy="0" iyz="0" izz="0" />
+    </inertial>
   </link>
   <joint name="wheel_right_joint" type="continuous">
@@ -134,15 +100,12 @@
         <mesh filename="package://servingbot_description/meshes/right_wheel.STL"/>
       </geometry>
-      <material
-        name="">
-        <color
-          rgba="0.79216 0.81961 0.93333 1" />
-      </material>
-    </visual>
-    <collision>
-      <origin xyz="0 0 0" rpy="0 0 0"/>
-      <geometry>
-        <mesh
-          filename="package://servingbot_description/meshes/right_wheel.STL" />
+      <material name="">
+        <color rgba="0.79216 0.81961 0.93333 1" />
+      </material>
+    </visual>
+    <collision>
+      <origin xyz="0 0 0" rpy="0 0 0"/>
+      <geometry>
+        <mesh filename="package://servingbot_description/meshes/right_wheel.STL" />
       </geometry>
     </collision>
@@ -150,8 +113,6 @@
       <origin xyz="0 -5.5511E-17 0" />
       <mass value="3.5" />
-      <inertia ixx="0" ixy="0" ixz="0"
-               iyy="0" iyz="0"
-               izz="0" />
-      </inertial>
+      <inertia ixx="0" ixy="0" ixz="0" iyy="0" iyz="0" izz="0" />
+    </inertial>
   </link>
   <joint name="caster_front_joint" type="fixed">
@@ -170,5 +131,5 @@
       <origin xyz="0 0.001 0" rpy="0 0 0"/>
       <geometry>
-	<cylinder length="0.050" radius="0.05"/>
+        <cylinder length="0.050" radius="0.05"/>
         <!--box size="0.050 0.090 0.010"/-->
       </geometry>
@@ -195,5 +156,5 @@
       <origin xyz="0 0.001 0" rpy="0 0 0"/>
       <geometry>
-	<cylinder length="0.050" radius="0.05"/>
+        <cylinder length="0.050" radius="0.05"/>
         <!--box size="0.050 0.090 0.010"/-->
       </geometry>
@@ -205,16 +166,9 @@
     </inertial>
   </link>
-  <joint
-    name="lidar_joint"
-    type="fixed">
-    <origin
-      xyz="0.23721 0 0.0453"
-      rpy="0 1.111E-15 0" />
-    <parent
-      link="base_link" />
-    <child
-      link="lidar_link" />
-    <axis
-      xyz="0 0 0" />
+  <joint name="lidar_joint" type="fixed">
+    <origin xyz="0.23721 0 0.0453" rpy="0 1.111E-15 0" />
+    <parent link="base_link" />
+    <child link="base_scan" />
+    <axis xyz="0 0 0" />
   </joint>
   <joint name="imu_joint" type="fixed">
@@ -224,41 +178,23 @@
   </joint>
   <link name="imu_link"/>
-  <link
-    name="lidar_link">
-    <inertial>
-      <origin
-        xyz="-0.25974 -0.001068 -0.098004"
-        rpy="0 0 3.141592" />
-      <mass
-        value="0.05" />
-      <inertia
-        ixx="6.003E-06"
-        ixy="2.5645E-07"
-        ixz="-2.0674E-06"
-        iyy="8.525E-06"
-        iyz="7.9724E-08"
-        izz="3.7518E-06" />
-    </inertial>
-    <visual>
-      <origin
-        xyz="0 0 0"
-        rpy="0 0 3.141592" />
-      <geometry>
-        <mesh
-          filename="package://servingbot_description/meshes/lidar.STL" />
-      </geometry>
-      <material
-        name="">
-        <color
-          rgba="0.79216 0.81961 0.93333 1" />
-      </material>
-    </visual>
-    <collision>
-      <origin
-        xyz="0 0 0"
-        rpy="0 0 0" />
-      <geometry>
-        <mesh
-          filename="package://servingbot_description/meshes/lidar.STL" />
+  <link name="base_scan">
+    <inertial>
+      <origin xyz="-0.25974 -0.001068 -0.098004" rpy="0 0 3.141592" />
+      <mass value="0.05" />
+      <inertia ixx="6.003E-06" ixy="2.5645E-07" ixz="-2.0674E-06" iyy="8.525E-06" iyz="7.9724E-08" izz="3.7518E-06" />
+    </inertial>
+    <visual>
+      <origin xyz="0 0 0" rpy="0 0 3.141592" />
+      <geometry>
+        <mesh filename="package://servingbot_description/meshes/lidar.STL" />
+      </geometry>
+      <material name="">
+        <color rgba="0.79216 0.81961 0.93333 1" />
+      </material>
+    </visual>
+    <collision>
+      <origin xyz="0 0 0" rpy="0 0 0" />
+      <geometry>
+        <mesh filename="package://servingbot_description/meshes/lidar.STL" />
       </geometry>
     </collision>

File: serving_mobile/servingbot_description/urdf/servingbot_rl.gazebo.xacro (robot description, xacro)
@@ -1,8 +1,9 @@
 <?xml version="1.0"?>
-<robot name="servingbot_sim" xmlns:xacro="http://ros.org/wiki/xacro">
+<robot name="servingbot_sim"
+  xmlns:xacro="http://ros.org/wiki/xacro">
   <xacro:arg name="laser_visual" default="false"/>
-  <xacro:arg name="imu_visual"   default="false"/>
-  <xacro:arg name="imu_visual"    default="false"/>
-  <xacro:arg name="lidar_visual"    default="true"/>
+  <xacro:arg name="imu_visual" default="false"/>
+  <xacro:arg name="imu_visual" default="false"/>
+  <xacro:arg name="lidar_visual" default="true"/>
   <gazebo reference="base_link">
     <material>Gazebo/DarkGrey</material>
@@ -37,5 +38,5 @@
     <material>Gazebo/FlatBlack</material>
   </gazebo>
-    <gazebo reference="caster_back_left_link">
+  <gazebo reference="caster_back_left_link">
     <mu1>0.1</mu1>
     <mu2>0.1</mu2>
@@ -111,5 +112,5 @@
     </plugin>
   </gazebo>
-  <gazebo reference="lidar_link">
+  <gazebo reference="base_scan">
     <material>Gazebo/FlatBlack</material>
     <sensor type="ray" name="lds_lfcd_sensor">
@@ -139,5 +140,5 @@
       <plugin name="gazebo_ros_lds_lfcd_controller" filename="libgazebo_ros_laser.so">
         <topicName>scan</topicName>
-        <frameName>lidar_link</frameName>
+        <frameName>base_scan</frameName>
       </plugin>
     </sensor>

File: serving_mobile/servingbot_description/urdf/servingbot_rl.urdf.xacro (robot description, xacro)
@@ -1,9 +1,10 @@
 <?xml version="1.0" ?>
-<robot name="servingbot" xmlns:xacro="http://ros.org/wiki/xacro">
+<robot name="servingbot"
+  xmlns:xacro="http://ros.org/wiki/xacro">
   <xacro:include filename="$(find servingbot_description)/urdf/common_properties.xacro"/>
   <xacro:include filename="$(find servingbot_description)/urdf/servingbot_rl.gazebo.xacro"/>
-<!-- base -->
-<link name="base_footprint"/>
- <joint name="base_joint" type="fixed">
+  <!-- base -->
+  <link name="base_footprint"/>
+  <joint name="base_joint" type="fixed">
     <parent link="base_footprint"/>
     <child link="base_link" />
@@ -19,5 +20,5 @@
     </visual>
     <collision>
-      <origin xyz="0 0.064  0.048" rpy="0 0 ${M_PI*0.5}"/>
+      <origin xyz="0 0.064  0.048" rpy="0 0 0"/>
       <geometry>
         <box size="0.265 0.265 0.089"/>
@@ -27,11 +28,9 @@
       <origin xyz="0 0.064 0.048" rpy="0 0 ${M_PI*0.5}"/>
       <mass value="0.01"/>
-      <inertia ixx="8.7002718e-03" ixy="-4.7576583e-05" ixz="1.1160499e-04"
-               iyy="8.6195418e-03" iyz="-3.5422299e-06"
-               izz="1.4612727e-02" />
+      <inertia ixx="8.7002718e-03" ixy="-4.7576583e-05" ixz="1.1160499e-04" iyy="8.6195418e-03" iyz="-3.5422299e-06" izz="1.4612727e-02" />
     </inertial>
   </link>
-<!-- body -->
- <link name="body_link">
+  <!-- body -->
+  <link name="body_link">
     <visual>
       <origin xyz="-0 0 0.2465" rpy="0 0 ${-M_PI*0.5}"/>
@@ -39,26 +38,17 @@
         <mesh filename="package://servingbot_description/meshes/base_plate.STL" />
       </geometry>
-      <material
-        name="">
-        <color
-          rgba="0.79216 0.81961 0.93333 1" />
+      <material name="">
+        <color rgba="0.79216 0.81961 0.93333 1" />
       </material>
     </visual>
   </link>
-  <joint
-    name="body_joint"
-    type="fixed">
-    <origin
-      xyz="0.0039057 0 -0.08"
-      rpy="-6.913E-15 -1.1102E-16 -5.4234E-31" />
-    <parent
-      link="base_link" />
-    <child
-      link="body_link" />
-    <axis
-      xyz="0 0 0" />
+  <joint name="body_joint" type="fixed">
+    <origin xyz="0.0039057 0 -0.08" rpy="-6.913E-15 -1.1102E-16 -5.4234E-31" />
+    <parent link="base_link" />
+    <child link="body_link" />
+    <axis xyz="0 0 0" />
   </joint>
-<!-- wheel -->
-<joint name="wheel_left_joint" type="continuous">
+  <!-- wheel -->
+  <joint name="wheel_left_joint" type="continuous">
     <parent link="base_link"/>
     <child link="wheel_left_link"/>
@@ -67,13 +57,11 @@
   </joint>
   <link name="wheel_left_link">
-     <visual>
+    <visual>
       <origin xyz="0 0 0" rpy="${-M_PI*0.5} 0 0"/>
       <geometry>
         <mesh filename="package://servingbot_description/meshes/left_wheel.STL"/>
       </geometry>
-      <material
-        name="">
-        <color
-          rgba="0.79216 0.81961 0.93333 1" />
+      <material name="">
+        <color rgba="0.79216 0.81961 0.93333 1" />
       </material>
     </visual>
@@ -87,8 +75,6 @@
       <origin xyz="0 0 0" />
       <mass value="2.8498940e-02" />
-      <inertia ixx="1.1175580e-05" ixy="-4.2369783e-11" ixz="-5.9381719e-09"
-               iyy="1.1192413e-05" iyz="-1.4400107e-11"
-               izz="2.0712558e-05" />
-      </inertial>
+      <inertia ixx="1.1175580e-05" ixy="-4.2369783e-11" ixz="-5.9381719e-09" iyy="1.1192413e-05" iyz="-1.4400107e-11" izz="2.0712558e-05" />
+    </inertial>
   </link>
   <joint name="wheel_right_joint" type="continuous">
@@ -104,8 +90,6 @@
         <mesh filename="package://servingbot_description/meshes/right_wheel.STL"/>
       </geometry>
-      <material
-        name="">
-        <color
-          rgba="0.79216 0.81961 0.93333 1" />
+      <material name="">
+        <color rgba="0.79216 0.81961 0.93333 1" />
       </material>
     </visual>
@@ -119,10 +103,8 @@
       <origin xyz="0 0 0" />
       <mass value="2.8498940e-02" />
-      <inertia ixx="1.1175580e-05" ixy="-4.2369783e-11" ixz="-5.9381719e-09"
-               iyy="1.1192413e-05" iyz="-1.4400107e-11"
-               izz="2.0712558e-05" />
-      </inertial>
+      <inertia ixx="1.1175580e-05" ixy="-4.2369783e-11" ixz="-5.9381719e-09" iyy="1.1192413e-05" iyz="-1.4400107e-11" izz="2.0712558e-05" />
+    </inertial>
   </link>
-<!-- caster -->
+  <!-- caster -->
   <joint name="caster_back_left_joint" type="fixed">
     <parent link="base_link"/>
@@ -140,7 +122,5 @@
       <origin xyz="0 0 0" />
       <mass value="0.005" />
-      <inertia ixx="0.001" ixy="0.0" ixz="0.0"
-               iyy="0.001" iyz="0.0"
-               izz="0.001" />
+      <inertia ixx="0.001" ixy="0.0" ixz="0.0" iyy="0.001" iyz="0.0" izz="0.001" />
     </inertial>
   </link>
@@ -160,7 +140,5 @@
       <origin xyz="0 0 0" />
       <mass value="0.005" />
-      <inertia ixx="0.001" ixy="0.0" ixz="0.0"
-               iyy="0.001" iyz="0.0"
-               izz="0.001" />
+      <inertia ixx="0.001" ixy="0.0" ixz="0.0" iyy="0.001" iyz="0.0" izz="0.001" />
     </inertial>
   </link>
@@ -180,10 +158,8 @@
       <origin xyz="0 0 0" />
       <mass value="0.005" />
-      <inertia ixx="0.001" ixy="0.0" ixz="0.0"
-               iyy="0.001" iyz="0.0"
-               izz="0.001" />
+      <inertia ixx="0.001" ixy="0.0" ixz="0.0" iyy="0.001" iyz="0.0" izz="0.001" />
     </inertial>
   </link>
-<!-- imu -->
+  <!-- imu -->
   <joint name="imu_joint" type="fixed">
     <parent link="base_link"/>
@@ -192,11 +168,11 @@
   </joint>
   <link name="imu_link"/>
-<!-- scan -->
+  <!-- scan -->
   <joint name="lidar_joint" type="fixed">
     <parent link="base_link"/>
-    <child link="lidar_link"/>
+    <child link="base_scan"/>
     <origin xyz="0 -0.235 0.29" rpy="0 0 ${-M_PI*0.5}"/>
   </joint>
-  <link name="lidar_link">
+  <link name="base_scan">
     <visual>
       <origin xyz="0 0 0" rpy="0 0 0"/>
@@ -204,8 +180,6 @@
         <mesh filename="package://servingbot_description/meshes/lidar.STL" />
       </geometry>
-      <material
-        name="">
-        <color
-          rgba="0.79216 0.81961 0.93333 1" />
+      <material name="">
+        <color rgba="0.79216 0.81961 0.93333 1" />
       </material>
     </visual>
